Commit message: modif coordonnées

File: urdf/robot_L.urdf (robot description, URDF)
Before this commit: robot robot_L, 2 links, 1 joints
Links:
- link base_link: geometry collision box size=0.2 0.2 0.2; visual box size=0.2 0.2 0.2
- link up_link: geometry collision box size=0.2 0.2 0.8; visual box size=0.2 0.2 0.8
