Commit message: adding new robots and envs

File: urdf/robot_chaine.urdf (robot description, URDF)
Before this commit: robot robot_L, 2 links, 1 joints
Links:
- added link tail_link; collision box size=0.4 0.4 1.6; visual box size=0.4 0.4 1.6
Joints:
- added joint up_to_tail: type revolute, parent up_link, child tail_link, origin xyz=0 0 0, axis 1 0 0, limit lower=-1.2 upper=1.2 effort=1000 velocity=0.5
