Commit message: nouveaux robots

File: urdf/robot_big_mesh.urdf (robot description, URDF)
Before this commit: robot robot_mesh, 1 links, 0 joints
Links:
- link base_link: geometry collision mesh filename=package://hpp_tutorial/meshes/big_pelvis.stl; visual mesh filename=package://hpp_tutorial/meshes/big_pelvis.stl

File: urdf/robot_cube_mesh.urdf (robot description, URDF)
Before this commit: robot robot_mesh, 1 links, 0 joints
Links:
- link base_link: geometry collision mesh filename=package://hpp_tutorial/meshes/cube.stl; visual mesh filename=package://hpp_tutorial/meshes/cube.stl

File: urdf/robot_siege.urdf (robot description, URDF)
Before this commit: robot robot_mesh, 1 links, 0 joints
Links:
- link base_link: geometry collision mesh filename=package://hpp_tutorial/meshes/siege.stl; visual mesh filename=package://hpp_tutorial/meshes/siege.stl

File: urdf/robot_strange.urdf (robot description, URDF)
Before this commit: robot robot_mesh, 1 links, 0 joints
Links:
- link base_link: geometry collision mesh filename=package://hpp_tutorial/meshes/strange.stl; visual mesh filename=package://hpp_tutorial/meshes/strange.stl
